Commit message: updated urdf with depth camera

File: go2_description/xacro/robot.xacro (robot description, xacro)
@@ -59,5 +59,5 @@
         <parent link="trunk"/>
         <child link="utlidar_lidar"/>
-        <origin rpy="0 -0.2 0" xyz="0.29515 -0.00003 -0.06597"/>
+        <origin rpy="0 -2.9415926 3.1415926" xyz="0.29515 -0.00003 -0.06597"/>
     </joint>
     <link name="utlidar_lidar">
@@ -103,4 +103,10 @@
     <link name="front_camera">
     </link>
+    <!-- Chassis Depth Camera -->
+    <xacro:include filename="$(find realsense2_description)/urdf/_d435i.urdf.xacro"/>
+    <xacro:sensor_d435i parent="trunk" name="d435i" use_nominal_extrinsics="true">
+        <origin xyz="0.32715 0.0 0.07" rpy="0.0 0.174533 0"/>
+        <!-- KRJ TODO: CHECK IF THIS IS CORRECT TRANSFORM. IS FROM CAD, SHOULD BE GOOD -->
+    </xacro:sensor_d435i>
     <!--
     <joint name="load_joint" type="fixed">

Commit message: changing lidar angle

File: go2_description/xacro/robot.xacro (robot description, xacro)
@@ -59,5 +59,8 @@
         <parent link="trunk"/>
         <child link="utlidar_lidar"/>
-        <origin rpy="0 -2.9415926 3.1415926" xyz="0.29515 -0.00003 -0.06597"/>
+        <!-- Calibrated against the D435 floor plane and depth (2026-10-20): mounted
+             upside down, pitched ~11.3 deg nose-down, ~2.5 deg roll. The previous
+             rpy="0 -2.9415926 3.1415926" had the pitch sign flipped (11.5 deg up). -->
+        <origin rpy="-3.0941 0.1969 0.0201" xyz="0.29515 -0.00003 -0.06597"/>
     </joint>
     <link name="utlidar_lidar">

Commit message: changed back lidar angle

File: go2_description/xacro/robot.xacro (robot description, xacro)
@@ -59,8 +59,5 @@
         <parent link="trunk"/>
         <child link="utlidar_lidar"/>
-        <!-- Calibrated against the D435 floor plane and depth (2026-10-20): mounted
-             upside down, pitched ~11.3 deg nose-down, ~2.5 deg roll. The previous
-             rpy="0 -2.9415926 3.1415926" had the pitch sign flipped (11.5 deg up). -->
-        <origin rpy="-3.0941 0.1969 0.0201" xyz="0.29515 -0.00003 -0.06597"/>
+        <origin rpy="0 -2.9415926 3.1415926" xyz="0.29515 -0.00003 -0.06597"/>
     </joint>
     <link name="utlidar_lidar">

Commit message: rotating lidar z axis

File: go2_description/xacro/robot.xacro (robot description, xacro)
@@ -59,5 +59,8 @@
         <parent link="trunk"/>
         <child link="utlidar_lidar"/>
-        <origin rpy="0 -2.9415926 3.1415926" xyz="0.29515 -0.00003 -0.06597"/>
+        <!-- Rotated 180 deg about the lidar's own z: its x axis points backward
+             (like Unitree's rpy="0 2.8782 0"). The previous "0 -2.9415926 3.1415926"
+             mirrored walls left/right and tilted the floor ~23 deg. -->
+        <origin rpy="0 2.9415926 0" xyz="0.29515 -0.00003 -0.06597"/>
     </joint>
     <link name="utlidar_lidar">

Commit message: added gps link

File: go2_description/xacro/robot.xacro (robot description, xacro)
@@ -74,4 +74,13 @@
     <link name="base_footprint">
     </link>
+    <!-- RTK GPS antenna (u-blox fixes are stamped frame_id "gps"): rigid on the
+         body, at the back edge of the trunk box, 2.5 in (0.0635 m) above its top -->
+    <joint name="gps_joint" type="fixed">
+        <parent link="trunk"/>
+        <child link="gps"/>
+        <origin rpy="0 0 0" xyz="${-trunk_length/2} 0 ${trunk_height/2 + 0.0635}"/>
+    </joint>
+    <link name="gps">
+    </link>
     <joint name="imu_joint" type="fixed">
         <parent link="trunk"/>
